File: pcb/main.brd (EAGLE design)
At the start: 49.2 x 30.5 mm, 5 parts

Commit message: pcb
Routing:
- net N$11: track 39.2 -> 37.7 mm
Changed lines of the file:
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@@
 <contactref element="JP_DISPLAY" pad="5"/>
 <contactref element="U$2" pad="4"/>
-<wire x1="8.69" y1="1.48" x2="3.81" y2="6.36" width="0.6" layer="16"/>
-<wire x1="3.81" y1="10.16" x2="3.81" y2="6.36" width="0.6" layer="16"/>
-<wire x1="17.92" y1="1.48" x2="8.69" y2="1.48" width="0.6" layer="16"/>
+<wire x1="11.23" y1="1.48" x2="3.81" y2="8.9" width="0.6" layer="16"/>
+<wire x1="3.81" y1="10.16" x2="3.81" y2="8.9" width="0.6" layer="16"/>
+<wire x1="17.92" y1="1.48" x2="11.23" y2="1.48" width="0.6" layer="16"/>
 <wire x1="27.67" y1="11.23" x2="17.92" y2="1.48" width="0.6" layer="16"/>
 <wire x1="33.02" y1="11.43" x2="32.82" y2="11.23" width="0.6" layer="16"/>
